File: BMS_Master.kicad_pcb (KiCad board)
At the start: 2 copper layers, 54 parts, among them J1 BMS_M_OUT, J2 BMS_M_IN, J3 PWR, J4 CAN, J5 PROG, SW1 SW_SPST, U1 STM32F103C8Tx, U2 AP2204K-ADJ, U3 AP2204K-ADJ, U4 SN65HVD256D, U5 BQ79600-Q1, Y1 32.768k, Y2 8M

Commit message: Finish schematic (For real), for basic requirements
Parts:
- added C24: 220n, Capacitor_SMD:C_0603_1608Metric, F.Cu at (105.7, 40.6)
- added D1: RUN_GREEN, LED_SMD:LED_0805_2012Metric, F.Cu at (36.2, 42.9)
- added H1: MountingHole_Pad, MountingHole:MountingHole_3.2mm_M3_ISO14580_Pad, F.Cu at (30.5, 44.9)
- added H2: MountingHole_Pad, MountingHole:MountingHole_3.2mm_M3_ISO14580_Pad, F.Cu at (30.5, 51.9)
- added H3: MountingHole_Pad, MountingHole:MountingHole_3.2mm_M3_ISO14580_Pad, F.Cu at (30.5, 59.0)
- added H4: MountingHole_Pad, MountingHole:MountingHole_3.2mm_M3_ISO14580_Pad, F.Cu at (30.5, 66.0)
- added R17: 10K, Resistor_SMD:R_0603_1608Metric, F.Cu at (101.5, 40.4)
- added R18: 10K, Resistor_SMD:R_0603_1608Metric, F.Cu at (101.5, 42.9)
- added R19: 100K, Resistor_SMD:R_0603_1608Metric, F.Cu at (101.5, 45.4)
- added R20: 1k, Resistor_SMD:R_0603_1608Metric, F.Cu at (36.0, 45.7)
- C1: footprint Package_SO:TSSOP-16-1EP_4.4x5mm_P0.65mm -> Capacitor_SMD:C_0603_1608Metric
- C10, C11, C12, C14, C15, C16, C17, C3, C5, C6, C7, C8, C9: footprint Capacitor_SMD:C_0805_2012Metric -> Capacitor_SMD:C_0603_1608Metric
- J3: footprint Connector_JST:JST_XH_S2B-XH-A_1x02_P2.50mm_Horizontal -> Connector_JST:JST_XH_B2B-XH-A_1x02_P2.50mm_Vertical
- J4, J5: footprint Connector_JST:JST_XH_S3B-XH-A_1x03_P2.50mm_Horizontal -> Connector_JST:JST_XH_B3B-XH-A_1x03_P2.50mm_Vertical
- R10: value 60R -> 100K
- R8, R9: value 60R -> 10K
- SW1: footprint Connector_JST:JST_XH_S2B-XH-A_1x02_P2.50mm_Horizontal -> Button_Switch_SMD:SW_SPST_FSMSM
- moved U5 3.30 mm to (66.7, 73.7)
- moved J3 1.91 mm to (108.3, 53.9)
Connections:
- C1 pad 1: +3V3 -> VIO
- C1 pad 2: GND -> SCLK
- C10 pad 2: GND -> SCLK
- C11 pad 2: GND -> SCLK
- C12 pad 2: GND -> SCLK
- C13 pad 1: GND -> SCLK
- C14 pad 1: GND -> SCLK
- C15 pad 1: GND -> SCLK
- C16 pad 1: Net-(U5-CVDD) -> +5V
- C16 pad 2: GND -> SCLK
- C17 pad 1: GND -> SCLK
- C17 pad 2: Net-(U5-DVDD) -> Net-(U5-VIO)
- C18 pad 2: GND1 -> SCLK
- C19 pad 2: GND1 -> SCLK
- C2 pad 1: +3V3 -> VIO
- C2 pad 2: GND -> SCLK
- C20 pad 2: GND1 -> SCLK
- C21 pad 2: GND1 -> SCLK
- C22 pad 2: GND1 -> SCLK
- C23 pad 2: GND1 -> SCLK
- C3 pad 1: GND -> SCLK
- C4 pad 1: GND -> SCLK
- C4 pad 2: +3V3 -> VIO
- C5 pad 1: +3V3 -> VIO
- C5 pad 2: GND -> SCLK
- C6 pad 1: +3V3 -> VIO
- C6 pad 2: GND -> SCLK
- C7 pad 1: +3V3 -> VIO
- C7 pad 2: GND -> SCLK
- C8 pad 1: +3V3 -> VIO
- C8 pad 2: GND -> SCLK
- C9 pad 2: GND -> SCLK
- J3 pad 2: GND -> SCLK
- J5 pad 3: GND -> SCLK
- R1 pad 1: +3V3 -> VIO
- R3 pad 1: GND -> SCLK
- R4 pad 1: GND -> SCLK
- R5 pad 2: +3V3 -> VIO
- SW1 pad 1: GND -> SCLK
- U1 pad 1: +3V3 -> VIO
- U1 pad 14: unconnected-(U1-PA4-Pad14) -> nCS
- U1 pad 15: unconnected-(U1-PA5-Pad15) -> SCLK
- U1 pad 16: unconnected-(U1-PA6-Pad16) -> MISO
- U1 pad 17: unconnected-(U1-PA7-Pad17) -> MOSI
- U1 pad 2: unconnected-(U1-PC13-Pad2) -> RUN_LED
- U1 pad 23: GND -> SCLK
- U1 pad 24: +3V3 -> VIO
- U1 pad 27: unconnected-(U1-PB14-Pad27) -> NFAULT
- U1 pad 28: unconnected-(U1-PB15-Pad28) -> SPI_RDY
- U1 pad 35: GND -> SCLK
- U1 pad 36: +3V3 -> VIO
- U1 pad 44: GND -> SCLK
- U1 pad 47: GND -> SCLK
- U1 pad 48: +3V3 -> VIO
- U1 pad 8: GND -> SCLK
- U1 pad 9: +3V3 -> VIO
- U2 pad 2: GND -> SCLK
- U3 pad 2: GND -> SCLK
- U3 pad 5: +3V3 -> VIO
- U4 pad 2: GND -> SCLK
- U4 pad 5: +3V3 -> VIO
- U5 pad 1: (no net) -> Net-(U5-VIO)
- U5 pad 10: (no net) -> COMLP
- U5 pad 11: (no net) -> COMLN
- U5 pad 12: (no net) -> COMHN
- U5 pad 13: (no net) -> COMHP
- U5 pad 14: (no net) -> +5V
- U5 pad 15: (no net) -> +5V
- U5 pad 16: (no net) -> +5V
- U5 pad 2: (no net) -> NFAULT
- U5 pad 3: (no net) -> VIO
- U5 pad 4: (no net) -> MOSI
- U5 pad 5: (no net) -> MISO
- U5 pad 6: (no net) -> Net-(U5-NFAULT)
- U5 pad 7: (no net) -> nCS
- U5 pad 8: (no net) -> SPI_RDY
- U5 pad 9: (no net) -> SCLK

Commit message: Initiate PCB layout and make some arrangement in Schematic
Parts:
- removed the C12 at (83.3, 57.9)
- added C12: 1u, Capacitor_SMD:C_0603_1608Metric, F.Cu at (133.4, 53.3)
- added C12: 100n, Capacitor_SMD:C_0603_1608Metric, F.Cu at (146.1, 79.3)
- added C25: 1u, Capacitor_SMD:C_0603_1608Metric, F.Cu at (68.0, 59.4)
- added D2: RUN_GREEN, LED_SMD:LED_0805_2012Metric, F.Cu at (102.0, 76.0)
- added D3: FAULT_RED, LED_SMD:LED_0805_2012Metric, F.Cu at (102.0, 79.0)
- added Q1: BC807, Package_TO_SOT_SMD:SOT-23, F.Cu at (71.8, 84.7)
- added R21: 60R, Resistor_SMD:R_0603_1608Metric, F.Cu at (76.0, 61.9)
- added R22: 60R, Resistor_SMD:R_0603_1608Metric, F.Cu at (76.0, 64.4)
- C1: value 100n -> 1u
- C10, C11, C9: value 20p -> 100n
- C13: value 10u -> 100n; footprint Capacitor_SMD:C_0805_2012Metric -> Capacitor_SMD:C_0603_1608Metric
- C14, C15: value 1u -> 220n
- C16, C17: value 220n -> 220p
- C22: value 220p -> 220n
- C23: value 220p -> 100n
- C24: value 220n -> 100n
- C3: value 1u -> 10u; footprint Capacitor_SMD:C_0603_1608Metric -> Capacitor_SMD:C_0805_2012Metric
- C5, C6, C7, C8: value 100n -> 20p
- D1: value RUN_GREEN -> PWR_Yellow
- J1: value BMS_M_OUT -> PWR; footprint Connector_Molex:Molex_Micro-Fit_3.0_43650-0200_1x02_P3.00mm_Horizontal -> Connector_JST:JST_XH_B2B-XH-A_1x02_P2.50mm_Vertical
- J2: value BMS_M_IN -> PROG; footprint Connector_Molex:Molex_Micro-Fit_3.0_43650-0200_1x02_P3.00mm_Horizontal -> Connector_JST:JST_XH_B3B-XH-A_1x03_P2.50mm_Vertical
- J3: value PWR -> BMS_M_OUT; footprint Connector_JST:JST_XH_B2B-XH-A_1x02_P2.50mm_Vertical -> Connector_Molex:Molex_Micro-Fit_3.0_43650-0200_1x02_P3.00mm_Horizontal
- J4: value CAN -> BMS_M_IN; footprint Connector_JST:JST_XH_B3B-XH-A_1x03_P2.50mm_Vertical -> Connector_Molex:Molex_Micro-Fit_3.0_43650-0200_1x02_P3.00mm_Horizontal
- J5: value PROG -> CAN
- R1: value 10k -> 1k
- R10: value 100K -> 1k
- R11, R20: value 1k -> 10K
- R12, R13: value 49R -> 10K
- R14, R15: value 49R -> 100K
- R16: value 1k -> 49R
- R17, R18: value 10K -> 49R
- R19: value 100K -> 49R
- R2: value 301k -> 100k
- R4: value 100k -> 301k
- R6: value 60R -> 10k
- R7: value 60R -> 1k
- R9: value 10K -> 1k
- U1: value STM32F103C8Tx -> AP2204K-ADJ; footprint Package_QFP:LQFP-48_7x7mm_P0.5mm -> Package_TO_SOT_SMD:SOT-23-5
- U3: value AP2204K-ADJ -> STM32F103C8Tx; footprint Package_TO_SOT_SMD:SOT-23-5 -> Package_QFP:LQFP-48_7x7mm_P0.5mm
- U4: value SN65HVD256D -> BQ79600-Q1; footprint Package_SO:SOIC-8_3.9x4.9mm_P1.27mm -> Package_SO:TSSOP-16_4.4x5mm_P0.65mm
- U5: value BQ79600-Q1 -> SN65HVD256D; footprint Package_SO:TSSOP-16_4.4x5mm_P0.65mm -> Package_SO:SOIC-8_3.9x4.9mm_P1.27mm
- Y1: value 32.768k -> 8M
- Y2: value 8M -> 32.768k
- moved R7 87.6 mm to (142.9, 72.4)
- moved C9 82.1 mm to (158.6, 81.5), turned to -90 degrees
- moved C10 81.1 mm to (154.9, 89.9), turned to 180 degrees
- moved U3 77.2 mm to (152.4, 83.8)
- moved D1 72.3 mm to (102.0, 72.9)
- moved C5 71.8 mm to (143.3, 86.4), turned to 180 degrees
- moved C11 70.3 mm to (150.5, 75.4)
- moved C13 67.8 mm to (146.4, 85.7), turned to 90 degrees
- moved SW1 67.4 mm to (64.5, 89.5)
- moved C6 66.0 mm to (139.9, 82.9), turned to 90 degrees
- moved J1 61.3 mm to (100.5, 85.6)
- moved U2 57.9 mm to (73.5, 94.0)
- moved Y1 56.0 mm to (142.8, 82.9)
- moved H3 55.3 mm to (81.6, 80.2)
- moved H1 55.3 mm to (81.6, 66.0)
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Connections:
- C1 pad 1: VIO -> GND
- C1 pad 2: SCLK -> +24V
- C10 pad 1: Net-(U1-PC15) -> VIO
- C10 pad 2: SCLK -> GND
- C11 pad 1: Net-(U1-PD0) -> VIO
- C11 pad 2: SCLK -> GND
- C13 pad 1: SCLK -> VIO
- C13 pad 2: +5V -> GND
- C14 pad 1: SCLK -> GND
- C14 pad 2: +24V -> VIO
- C15 pad 1: SCLK -> GND
- C15 pad 2: Net-(C15-Pad2) -> Net-(U4-DVDD)
- C16 pad 1: +5V -> COMHP
- C16 pad 2: SCLK -> GND
- C17 pad 1: SCLK -> COMHN
- C17 pad 2: Net-(U5-VIO) -> GND
- C18 pad 2: SCLK -> GND
- C19 pad 2: SCLK -> GND
- C2 pad 1: VIO -> GND
- C2 pad 2: SCLK -> +5V
- C20 pad 2: SCLK -> GND
- C21 pad 2: SCLK -> GND
- C22 pad 1: COMHP -> +5V
- C22 pad 2: SCLK -> GND
- C23 pad 1: COMHN -> GND
- C23 pad 2: SCLK -> +5V
- C24 pad 1: SCLK -> GND
- C3 pad 1: SCLK -> GND
- C4 pad 1: SCLK -> GND
- C5 pad 1: VIO -> Net-(U3-PD0)
- C5 pad 2: SCLK -> GND
- C6 pad 1: VIO -> Net-(U3-PD1)
- C6 pad 2: SCLK -> GND
- C7 pad 1: VIO -> Net-(U3-PC14)
- C7 pad 2: SCLK -> GND
- C8 pad 1: VIO -> Net-(U3-PC15)
- C8 pad 2: SCLK -> GND
- C9 pad 1: Net-(U1-PC14) -> VIO
- C9 pad 2: SCLK -> GND
- D1 pad 1: SCLK -> GND
- H1 pad 1: SCLK -> GND
- H2 pad 1: SCLK -> GND
- H3 pad 1: SCLK -> GND
- H4 pad 1: SCLK -> GND
- J1 pad 1: Net-(J1-Pin_1) -> +24V
- J1 pad 2: Net-(J1-Pin_2) -> GND
- J2 pad 1: Net-(J2-Pin_1) -> SWDIO
- J2 pad 2: Net-(J2-Pin_2) -> SWCLK
- J3 pad 1: +24V -> Net-(J3-Pin_1)
- J3 pad 2: SCLK -> Net-(J3-Pin_2)
- J4 pad 1: CAN_N -> Net-(J4-Pin_1)
- J4 pad 2: unconnected-(J4-Pin_2-Pad2) -> Net-(J4-Pin_2)
- J5 pad 1: SWDIO -> CAN_N
- J5 pad 2: SWCLK -> unconnected-(J5-Pin_2-Pad2)
- J5 pad 3: SCLK -> CAN_P
- R1 pad 1: VIO -> Net-(D1-A)
- R1 pad 2: Net-(SW1-B) -> VIO
- R10 pad 1: VIO -> COMLP
- R10 pad 2: NFAULT -> COMLN
- R11 pad 1: COMLP -> VIO
- R11 pad 2: COMLN -> MOSI
- R12 pad 1: COMLP -> VIO
- R12 pad 2: Net-(R12-Pad2) -> MISO
- R13 pad 1: COMLN -> VIO
- R13 pad 2: Net-(R13-Pad2) -> nCS
- R14 pad 1: COMHP -> VIO
- R14 pad 2: Net-(R14-Pad2) -> SPI_RDY
- R15 pad 1: COMHN -> VIO
- R15 pad 2: Net-(R15-Pad2) -> NFAULT
- R16 pad 2: COMHN -> Net-(R16-Pad2)
- R17 pad 1: Net-(U5-NFAULT) -> COMHN
- R17 pad 2: SCLK -> Net-(R17-Pad2)
- R18 pad 1: VIO -> COMLP
- R18 pad 2: nCS -> Net-(R18-Pad2)
- R19 pad 1: VIO -> COMLN
- R19 pad 2: SPI_RDY -> Net-(R19-Pad2)
- R2 pad 1: Net-(U2-ADJ) -> GND
- R2 pad 2: +5V -> Net-(U1-ADJ)
- R20 pad 1: Net-(D1-A) -> Net-(Q1-B)
- R20 pad 2: RUN_LED -> BMS_FAULT
- R3 pad 1: SCLK -> GND
- R4 pad 1: SCLK -> Net-(U1-ADJ)
- R4 pad 2: Net-(U3-ADJ) -> +5V
- R5 pad 1: Net-(U3-ADJ) -> Net-(U2-ADJ)
- R6 pad 1: Net-(C15-Pad2) -> VIO
- R6 pad 2: CAN_P -> Net-(SW1-B)
- R7 pad 1: CAN_N -> Net-(D2-A)
- R7 pad 2: Net-(C15-Pad2) -> RUN_LED
- R8 pad 1: VIO -> SCLK
- R8 pad 2: MOSI -> GND
- R9 pad 1: VIO -> COMHP
- R9 pad 2: MISO -> COMHN
- SW1 pad 1: SCLK -> GND
- TR1 pad 1: Net-(R14-Pad2) -> Net-(R16-Pad2)
- TR1 pad 3: Net-(R15-Pad2) -> Net-(R17-Pad2)
- TR1 pad 4: Net-(J1-Pin_2) -> Net-(J3-Pin_2)
- TR1 pad 6: Net-(J1-Pin_1) -> Net-(J3-Pin_1)
- TR2 pad 1: Net-(R12-Pad2) -> Net-(R18-Pad2)
- TR2 pad 3: Net-(R13-Pad2) -> Net-(R19-Pad2)
- TR2 pad 4: Net-(J2-Pin_2) -> Net-(J4-Pin_2)
- TR2 pad 6: Net-(J2-Pin_1) -> Net-(J4-Pin_1)
- U1 pad 1: VIO -> +24V
- U1 pad 2: RUN_LED -> GND
- U1 pad 3: Net-(U1-PC14) -> +24V
- U1 pad 4: Net-(U1-PC15) -> Net-(U1-ADJ)
- U1 pad 5: Net-(U1-PD0) -> +5V
- U2 pad 1: +24V -> +5V
- U2 pad 2: SCLK -> GND
- U2 pad 3: +24V -> +5V
- U2 pad 5: +5V -> VIO
- U3 pad 1: +5V -> VIO
- U3 pad 2: SCLK -> RUN_LED
- U3 pad 3: +5V -> Net-(U3-PC14)
- U3 pad 4: Net-(U3-ADJ) -> Net-(U3-PC15)
- U3 pad 5: VIO -> Net-(U3-PD0)
- U4 pad 1: CAN_RX -> Net-(U4-DVDD)
- U4 pad 2: SCLK -> NFAULT
- U4 pad 3: +5V -> VIO
- U4 pad 4: CAN_TX -> MOSI
- U4 pad 5: VIO -> MISO
- U4 pad 6: CAN_N -> SCLK
- U4 pad 7: CAN_P -> nCS
- U4 pad 8: unconnected-(U4-S-Pad8) -> SPI_RDY
- U5 pad 1: Net-(U5-VIO) -> CAN_RX
- U5 pad 2: NFAULT -> GND
- U5 pad 3: VIO -> +5V
- U5 pad 4: MOSI -> CAN_TX
- U5 pad 5: MISO -> VIO
- U5 pad 6: Net-(U5-NFAULT) -> CAN_N
- U5 pad 7: nCS -> CAN_P
- U5 pad 8: SPI_RDY -> unconnected-(U5-S-Pad8)
- Y1 pad 1: Net-(U1-PC14) -> Net-(U3-PD1)
- Y1 pad 2: Net-(U1-PC15) -> GND
- Y1 pad 3: (no net) -> Net-(U3-PD0)
- Y1 pad 4: (no net) -> GND
- Y2 pad 1: Net-(U1-PD0) -> Net-(U3-PC15)
- Y2 pad 2: Net-(U1-PD1) -> GND
- Y2 pad 3: (no net) -> Net-(U3-PC14)
- Y2 pad 4: (no net) -> GND
Other:
- rule pad_to_mask_clearance: 0 -> 0.08

Commit message: Finish PCB layout Ver 1.0
Parts:
- removed the C12 at (133.4, 53.3)
- added G***: LOGO, Logos:fsae_logo, F.Cu at (116.1, 79.0)
- added kibuzzard-6797B0CB: G***, kibuzzard-6797B0CB, F.Cu at (73.2, 44.6)
- added kibuzzard-6797B107: G***, kibuzzard-6797B107, F.Cu at (91.5, 75.5)
- added kibuzzard-6797B129: G***, kibuzzard-6797B129, F.Cu at (73.0, 48.1)
- added kibuzzard-6797B18E: G***, kibuzzard-6797B18E, F.Cu at (78.5, 40.6)
- added kibuzzard-6797B1AA: G***, kibuzzard-6797B1AA, F.Cu at (94.4, 40.7)
- added kibuzzard-6797B21F: G***, kibuzzard-6797B21F, F.Cu at (78.6, 81.1)
- added kibuzzard-6797B237: G***, kibuzzard-6797B237, F.Cu at (70.2, 67.8)
- added kibuzzard-6797BA30: G***, kibuzzard-6797BA30, F.Cu at (98.2, 54.1)
- added kibuzzard-6797BA57: G***, kibuzzard-6797BA57, F.Cu at (127.2, 58.8)
- added kibuzzard-6797BA64: G***, kibuzzard-6797BA64, F.Cu at (127.4, 72.2)
- added kibuzzard-6797C095: G***, kibuzzard-6797C095, F.Cu at (115.7, 40.8)
- J2: footprint Connector_JST:JST_XH_B3B-XH-A_1x03_P2.50mm_Vertical -> Connector_PinHeader_2.54mm:PinHeader_1x03_P2.54mm_Vertical
- moved Y1 72.4 mm to (74.8, 58.0)
- moved C9 72.4 mm to (91.2, 55.1)
- moved C6 72.4 mm to (72.0, 58.0)
- moved C11 72.1 mm to (82.4, 51.8), turned to 90 degrees
- moved C13 72.0 mm to (78.2, 62.5), turned to -90 degrees
- moved C10 71.8 mm to (87.7, 64.6)
- moved U3 71.8 mm to (85.2, 58.5)
- moved Y2 71.3 mm to (76.0, 54.0)
- moved C5 71.2 mm to (77.7, 58.8), turned to -90 degrees
- moved C12 70.3 mm to (80.9, 53.0)
- moved H4 67.4 mm to (129.9, 40.3)
- moved R7 66.6 mm to (80.2, 49.9)
- moved J5 53.4 mm to (83.8, 40.2)
- moved H3 48.4 mm to (129.9, 78.8)
- moved C20 47.0 mm to (107.0, 53.0), turned to 180 degrees
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Connections:
- J5 pad 1: CAN_N -> CAN_P
- J5 pad 3: CAN_P -> CAN_N
- TR2 pad 1: Net-(R18-Pad2) -> Net-(R19-Pad2)
- TR2 pad 3: Net-(R19-Pad2) -> Net-(R18-Pad2)
- TR2 pad 4: Net-(J4-Pin_2) -> Net-(J4-Pin_1)
- TR2 pad 6: Net-(J4-Pin_1) -> Net-(J4-Pin_2)
Routing:
- net VIO: track 0.00 -> 139.8 mm, vias 0 -> 6
- net GND: track 0.00 -> 66.9 mm, vias 0 -> 10
- net +5V: track 0.00 -> 63.0 mm, vias 0 -> 4
- net BMS_FAULT: track 0.00 -> 30.0 mm, vias 0 -> 2
- net nCS: track 0.00 -> 27.9 mm, vias 0 -> 2
- net SCLK: track 0.00 -> 25.8 mm, vias 0 -> 2
- net MISO: track 0.00 -> 24.0 mm, vias 0 -> 2
- net MOSI: track 0.00 -> 23.0 mm, vias 0 -> 2
- net NFAULT: track 0.00 -> 22.4 mm, vias 0 -> 2
- net COMHP: track 0.00 -> 22.1 mm
- net COMHN: track 0.00 -> 21.6 mm
- net SPI_RDY: track 0.00 -> 18.2 mm
- net Net-(C25-Pad2): track 0.00 -> 12.8 mm
- net CAN_P: track 0.00 -> 12.0 mm
- net Net-(U1-ADJ): track 0.00 -> 11.9 mm
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- added copper zone on B.Cu, net GND
- added copper zone on F.Cu, net GND
Other:
- board outline added: 65 x 45 mm
