File: BMS_Master.kicad_sch (KiCad schematic)
At the start: 79 parts, among them J1 PWR, J2 PROG, J3 BMS_M_OUT, J4 BMS_M_IN, J5 CAN, J6 Current_Sensor, Q1 BC807, SW1 SW_SPST, U1 AP2204K-ADJ, U2 AP2204K-ADJ, U3 STM32F103C8Tx, U4 BQ79600-Q1, U5 SN65HVD256D, Y1 8M, Y2 32.768k

Commit message: Finish layout ver 1, already abandoned
Parts:
- J6: footprint (none) -> Connector_JST:JST_XH_B4B-XH-A_1x04_P2.50mm_Vertical
Changed lines of the file:
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@@
       (effects (font (size 1.27 1.27)) (justify left))
     )
-    (property "Footprint" "" (at 80.645 161.29 0)
+    (property "Footprint" "Connector_JST:JST_XH_B4B-XH-A_1x04_P2.50mm_Vertical" (at 80.645 161.29 0)
       (effects (font (size 1.27 1.27)) hide)
     )
